File: Devboard-PCB/Devboard.kicad_pcb (KiCad board)
At the start: 2 copper layers, 39.3 x 51.7 mm, 45 parts, among them J1 USB_C_Receptacle_USB2.0_14P, J2 Conn_01x20, J3 Conn_01x20, J4 Conn_01x03, SW1 SW_Push, SW2 SW_Push, U1 RP2040, U2 MCP1700x-120xxMB, U3 W25Q128JVS, U4 ER_OLEDM0.91_1x-I2C, U5 TPS63000, Y2 Crystal_GND24

Commit message: Worked on replacing the 0201 capacitors with 0402 and 0603 caps
Parts:
- C1, C10, C11, C12, C13, C14, C15, C16, C17, C19, C2, C3, C4, C5, C6, C7, C8: footprint Capacitor_SMD:C_0201_0603Metric -> Capacitor_SMD:C_0402_1005Metric_Pad0.74x0.62mm_HandSolder
- C18, C20, C21, C9: footprint Capacitor_SMD:C_0201_0603Metric -> Capacitor_SMD:C_0603_1608Metric_Pad1.08x0.95mm_HandSolder
- moved C9 2.05 mm to (160.1, 64.7)
- moved C7 1.61 mm to (159.8, 66.3)
- moved C19 1.00 mm to (175.3, 53.6), turned to 90 degrees
- moved C21 0.54 mm to (169.9, 49.0)
- moved C5 0.49 mm to (160.9, 72.3)
- moved C11 0.46 mm to (157.2, 64.1)
- moved C12 0.30 mm to (153.7, 64.3)
- moved C6 0.20 mm to (156.0, 64.3)
- moved C2 0.19 mm to (149.9, 68.6)
- moved C4 0.16 mm to (157.9, 66.4)
- moved C8 0.15 mm to (160.5, 68.7)
- moved C1 0.14 mm to (155.3, 77.5)
Routing:
- net +3V3: track 211.3 -> 276.7 mm
- net Net-(U1-USB_DP): track 11.7 -> 13.4 mm, vias 0 -> 2
- net GND: track 135.9 -> 137.5 mm
- net Net-(U5-L2): track 10.5 -> 11.6 mm
- net GPIO9: track 12.9 -> 13.9 mm
- net Net-(U5-EN): track 7.01 -> 7.96 mm
- net Net-(U1-USB_DM): track 11.4 -> 12.1 mm, vias 0 -> 2
